Commit message: after reinstallation, Gazebo crashes occasionally, not able to receive camera data

File: turtlebot2i/src/turtlebot2i_description/urdf/sensors/sr300.urdf.xacro (robot description, xacro)
@@ -68,5 +68,5 @@
     -->
     <joint name="camera_sr300_depth_joint" type="fixed">
-        <origin xyz="0 ${sr300_cam_depth_offset} 0" rpy="0 -1.16 0" />
+        <origin xyz="0 ${sr300_cam_depth_offset} 0" rpy="0 0 0" />
         <parent link="camera_sr300_rgb_frame" />
         <child link="camera_sr300_depth_frame" />

File: turtlebot2i/src/turtlebot2i_description/urdf/turtlebot_gazebo.urdf.xacro (robot description, xacro)
@@ -5,5 +5,5 @@
         <robotNamespace>/turtlebot</robotNamespace>
         <robotSimType>gazebo_ros_control/DefaultRobotHWSim</robotSimType>
-        <legacyModeNS>true</legacyModeNS>
+	<legacyModeNS>true</legacyModeNS>
     </plugin>
   </gazebo>

Commit message: reconstructed from start, able to see camera image and teleop, the arm doesn't move, haven't started mapping configuretion

File: turtlebot2i/src/turtlebot2i_description/urdf/sensors/sr300.urdf.xacro (robot description, xacro)
@@ -68,5 +68,5 @@
     -->
     <joint name="camera_sr300_depth_joint" type="fixed">
-        <origin xyz="0 ${sr300_cam_depth_offset} 0" rpy="0 0 0" />
+        <origin xyz="0 ${sr300_cam_depth_offset} 0" rpy="0 -1.16 0" />
         <parent link="camera_sr300_rgb_frame" />
         <child link="camera_sr300_depth_frame" />

File: turtlebot2i/src/turtlebot2i_description/urdf/turtlebot_gazebo.urdf.xacro (robot description, xacro)
@@ -5,5 +5,5 @@
         <robotNamespace>/turtlebot</robotNamespace>
         <robotSimType>gazebo_ros_control/DefaultRobotHWSim</robotSimType>
-	<legacyModeNS>true</legacyModeNS>
+        <legacyModeNS>true</legacyModeNS>
     </plugin>
   </gazebo>
