Commit message: able to control gripper and get their transformation, rtabmap images turn red, wheels still missing

File: turtlebot2i/src/phantomx_pincher_arm/phantomx_pincher_arm_description/urdf/phantomx_pincher_arm.xacro (robot description, xacro)
@@ -16,5 +16,5 @@
       <type>transmission_interface/SimpleTransmission</type>
       <joint name="arm_shoulder_pan_joint">
-        <hardwareInterface>EffortJointInterface</hardwareInterface>
+        <hardwareInterface>hardware_interface/EffortJointInterface</hardwareInterface>
       </joint>
       <actuator name="arm_shoulder_pan_actuator">
@@ -31,5 +31,5 @@
       <type>transmission_interface/SimpleTransmission</type>
       <joint name="arm_bicep_joint">
-        <hardwareInterface>EffortJointInterface</hardwareInterface>
+        <hardwareInterface>hardware_interface/EffortJointInterface</hardwareInterface>
       </joint>
       <actuator name="arm_bicep_actuator">
@@ -46,5 +46,5 @@
       <type>transmission_interface/SimpleTransmission</type>
       <joint name="arm_forearm_joint">
-        <hardwareInterface>EffortJointInterface</hardwareInterface>
+        <hardwareInterface>hardware_interface/EffortJointInterface</hardwareInterface>
       </joint>
       <actuator name="arm_forearm_actuator">
@@ -61,5 +61,5 @@
       <type>transmission_interface/SimpleTransmission</type>
       <joint name="arm_wrist_flex_joint">
-        <hardwareInterface>EffortJointInterface</hardwareInterface>
+        <hardwareInterface>hardware_interface/EffortJointInterface</hardwareInterface>
       </joint>
       <actuator name="arm_wrist_flex_actuator">
@@ -71,5 +71,5 @@
   <xacro:include filename="$(find phantomx_pincher_arm_description)/urdf/phantomx_pincher_gripper.xacro"/>
 <!-- gripper_link -->
-    <link name="gripper_link"/>
+    <!--link name="gripper_link"/>
     <joint name="gripper_link_joint" type="revolute">
       <origin xyz="0.110 0 0" rpy="0 0 0"/>
@@ -79,4 +79,18 @@
       <axis xyz="1 0 0"/>
     </joint>
+    <transmission name="gripper_link_transmission">
+      <type>transmission_interface/SimpleTransmission</type>
+      <joint name="gripper_link_joint">
+        <hardwareInterface>hardware_interface/EffortJointInterface</hardwareInterface>
+      </joint>
+      <actuator name="gripper_link_actuator">
+        <hardwareInterface>EffortJointInterface</hardwareInterface>
+        <mechanicalReduction>1</mechanicalReduction>
+      </actuator>
+    </transmission>
+    <gazebo reference="gripper_link">
+      <material>Gazebo/${color}</material>
+      <gravity>true</gravity>
+    </gazebo-->
   <!--gazebo>
       <gripper name="gripper">

File: turtlebot2i/src/phantomx_pincher_arm/phantomx_pincher_arm_description/urdf/phantomx_pincher_gripper.xacro (robot description, xacro)
@@ -7,18 +7,29 @@
       <origin xyz="0.070 0 0" rpy="0 0 0"/>
       <axis xyz="0 1 0"/>
-      <limit effort="30" velocity="0.5" lower="0.002" upper="0.032"/>
+      <limit effort="3" velocity="0.05" lower="0.002" upper="0.032"/>
       <parent link="arm_wrist_flex_link"/>
       <child link="gripper_active_link"/>
+      <dynamics friction="0.13"/>
     </joint>
     <pincher_finger name="gripper_active" color="${color}" >
       <origin xyz="0 0 0" rpy="0 0 0"/>
     </pincher_finger>
+    <transmission name="gripper_joint_transmission">
+      <type>transmission_interface/SimpleTransmission</type>
+      <joint name="gripper_joint">
+        <hardwareInterface>hardware_interface/EffortJointInterface</hardwareInterface>
+      </joint>
+      <actuator name="gripper_joint_actuator">
+        <hardwareInterface>EffortJointInterface</hardwareInterface>
+        <mechanicalReduction>1</mechanicalReduction>
+      </actuator>
+    </transmission>
     <!-- Finger 2 -->
     <!-- Note: currently static but should be a Mimic of Finger 1 -->
-    <joint name="gripper2_joint" type="fixed">
+    <!--joint name="gripper2_joint" type="fixed">
       <origin xyz="0.070 -0.016 0" rpy="0 0 0"/>
       <parent link="arm_wrist_flex_link"/>
       <child link="gripper_active2_link"/>
-    </joint>
+    </joint-->
     <pincher_finger name="gripper_active2" color="${color}" >
       <origin xyz="0 0 0" rpy="${M_PI} 0 0"/>
@@ -26,12 +37,23 @@
     <!-- Using Mimic -->
     <!-- gripper 2 joint -->
-    <!--  TODO: Test Mimic ->
+    <!--  TODO: Test Mimic -->
     <joint name="gripper2_joint" type="prismatic">
       <origin xyz="0.070 0 0" rpy="0 0 0"/>
       <axis xyz="0 1 0"/>
-      <limit effort="30" velocity="0.5" lower="-0.016" upper="-0.002"/>
+      <limit effort="3" velocity="0.05" lower="-0.032" upper="-0.002"/>
       <parent link="arm_wrist_flex_link"/>
       <child link="gripper_active2_link"/>
-      <mimic joint="gripper_joint" multiplier="-1"  offset = "0"/>
-    </joint-->
+      <!--mimic joint="gripper_joint" multiplier="-1"  offset = "0"/-->
+      <dynamics friction="0.13"/>
+    </joint>
+    <transmission name="gripper2_joint_transmission">
+      <type>transmission_interface/SimpleTransmission</type>
+      <joint name="gripper2_joint">
+        <hardwareInterface>hardware_interface/EffortJointInterface</hardwareInterface>
+      </joint>
+      <actuator name="gripper2_joint_actuator">
+        <hardwareInterface>EffortJointInterface</hardwareInterface>
+        <mechanicalReduction>1</mechanicalReduction>
+      </actuator>
+    </transmission>
 </robot>

Commit message: modified URDFs and launches to use MoveIt plugin in RVIZ

File: turtlebot2i/src/phantomx_pincher_arm/phantomx_pincher_arm_description/urdf/phantomx_pincher_arm.xacro (robot description, xacro)
@@ -71,5 +71,5 @@
   <xacro:include filename="$(find phantomx_pincher_arm_description)/urdf/phantomx_pincher_gripper.xacro"/>
 <!-- gripper_link -->
-    <!--link name="gripper_link"/>
+    <link name="gripper_link"/>
     <joint name="gripper_link_joint" type="revolute">
       <origin xyz="0.110 0 0" rpy="0 0 0"/>
@@ -79,5 +79,5 @@
       <axis xyz="1 0 0"/>
     </joint>
-    <transmission name="gripper_link_transmission">
+    <!--transmission name="gripper_link_transmission">
       <type>transmission_interface/SimpleTransmission</type>
       <joint name="gripper_link_joint">
