Commit message: Updated moveit configs and removed second gripper for simplicity

File: turtlebot2i/src/phantomx_pincher_arm/phantomx_pincher_arm_description/urdf/phantomx_pincher_gripper.xacro (robot description, xacro)
@@ -27,9 +27,9 @@
     <!-- Finger 2 -->
     <!-- Note: currently static but should be a Mimic of Finger 1 -->
-    <!--joint name="gripper2_joint" type="fixed">
+    <joint name="gripper2_joint" type="fixed">
       <origin xyz="0.070 -0.016 0" rpy="0 0 0"/>
       <parent link="arm_wrist_flex_link"/>
       <child link="gripper_active2_link"/>
-    </joint-->
+    </joint>
     <pincher_finger name="gripper_active2" color="${color}" >
       <origin xyz="0 0 0" rpy="${M_PI} 0 0"/>
@@ -38,5 +38,5 @@
     <!-- gripper 2 joint -->
     <!--  TODO: Test Mimic -->
-    <joint name="gripper2_joint" type="prismatic">
+    <!--joint name="gripper2_joint" type="prismatic">
       <origin xyz="0.070 0 0" rpy="0 0 0"/>
       <axis xyz="0 1 0"/>
@@ -44,5 +44,4 @@
       <parent link="arm_wrist_flex_link"/>
       <child link="gripper_active2_link"/>
-      <!--mimic joint="gripper_joint" multiplier="-1"  offset = "0"/-->
       <dynamics friction="0.13"/>
     </joint>
@@ -56,4 +55,4 @@
         <mechanicalReduction>1</mechanicalReduction>
       </actuator>
-    </transmission>
+    </transmission-->
 </robot>

File: turtlebot2i/src/turtlebot2i_description/urdf/sensors/sr300.urdf.xacro (robot description, xacro)
@@ -53,5 +53,5 @@
     -->
     <joint name="camera_sr300_rgb_joint" type="fixed">
-      <origin xyz="${sr300_cam_rgb_px} ${sr300_cam_rgb_py} ${sr300_cam_rgb_pz}" rpy="0 1.16 0"/>
+      <origin xyz="${sr300_cam_rgb_px} ${sr300_cam_rgb_py} ${sr300_cam_rgb_pz}" rpy="0 0 0"/>
       <parent link="camera_sr300"/>
       <child link="camera_sr300_rgb_frame" />
@@ -68,5 +68,5 @@
     -->
     <joint name="camera_sr300_depth_joint" type="fixed">
-        <origin xyz="0 ${sr300_cam_depth_offset} 0" rpy="0 -1.16 0" />
+        <origin xyz="0 ${sr300_cam_depth_offset} 0" rpy="0 0 0" />
         <parent link="camera_sr300_rgb_frame" />
         <child link="camera_sr300_depth_frame" />
